File: hardware/cartucho/vet3000_cartucho.kicad_pcb (KiCad board)
At the start: 2 copper layers, 72 x 60 mm, 13 parts, among them J1 CN1 VET 3000 (soquete de bord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, J2 EXP, U1 27C128, U2 74HCT00

Commit message: Cartucho: hardware sob CERN-OHL-S-2.0 e passo de 2,54 mm confirmado
- hardware/cartucho/ passa a ser licenciado sob a CERN-OHL-S-2.0 (LICENSE
  com o texto oficial, nota de licença e Source Location no README, nos
  cabeçalhos dos scripts, no bloco de título e na serigrafia do verso).
  O restante do repositório continua sob a GPL-3.0-or-later.
- Passo dos dedos do CN1 medido no aparelho: 2,54 mm (o do footprint).
- Gerbers, PDF e renders regenerados; ERC/DRC/paridade sem problemas.

Co-Authored-By: Claude Opus 5.5 <noreply@anthropic.com>
Other:
- board text added: "(c) 2026 Leonardo Roman da Rosa - CERN-OHL-S-2.0"
- board text added: "github.com/lrrosa/vet3000"
- board text removed: "(c) 2026 Leonardo Roman da Rosa - GPL-3.0 - github.com/lrrosa/vet3000"
Changed lines of the file:
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@@
 	)
 	(paper "A4")
+	(title_block
+		(title "VET 3000 - Cartucho de ROM (CN1)")
+		(date "2026-09-27")
+		(rev "1.0")
+		(company "Leonardo Roman da Rosa")
+		(comment 1 "Copyright (C) 2026 Leonardo Roman da Rosa - CERN-OHL-S-2.0")
+		(comment 2 "Source location: https://github.com/lrrosa/vet3000")
+	)
 	(layers
 		(0 "F.Cu" signal)
@@
 		)
 	)
-	(gr_text "(c) 2026 Leonardo Roman da Rosa - GPL-3.0 - github.com/lrrosa/vet3000"
+	(gr_text "github.com/lrrosa/vet3000"
+		(at 136 128.699999 0)
+		(layer "B.SilkS")
+		(effects
+			(font
+				(size 0.8 0.8)
+				(thickness 0.12)
+			)
+			(justify mirror)
+		)
+	)
+	(gr_text "(c) 2026 Leonardo Roman da Rosa - CERN-OHL-S-2.0"
 		(at 136 146.3 0)
 		(layer "B.SilkS")
@@
 	)
 	(gr_text "cartucho de ROM - conector CN1"
-		(at 136 135.6 0)
+		(at 136 135.7 0)
 		(layer "B.SilkS")
 		(effects
@@
 	)
 	(gr_text "ESTE LADO PARA FORA"
-		(at 136 138.9 0)
+		(at 136 139 0)
 		(layer "B.SilkS")
 		(effects
@@
 	)
 	(gr_text "VET 3000"
-		(at 136 131.5 0)
+		(at 136 132 0)
 		(layer "B.SilkS")
 		(effects
 			(font
-				(size 3 3)
-				(thickness 0.6)
+				(size 2.6 2.6)
+				(thickness 0.52)
 				(bold yes)
 			)
