File: hardware/placa-principal/vet3000_placa.kicad_sch (KiCad schematic)
At the start: 0 parts

Commit message: Esquema: placa da fonte e medidas do teclado, pull-ups e /OE
- Folha Fonte (fonte.kicad_sch), levantada das fotos dos dois lados da
  placa: ponte com derivação central, 7805, 7812, 7905 com bomba de carga,
  backup da RAM (+3V_BAT) e conector de saída. Explica os ~11 V no +5 V
  quando a fonte é testada sem carga.
- Teclado medido: U16 (74LS273) e U22 (74LS244) ligam D0-D7 com os mesmos
  pinos da revista (Fig. 14), e o /CLR do U16 vai ao +5 V. O conector das
  membranas é o CN3: pino 1 embaixo à esquerda, ímpares = membrana inferior
  (linhas, U16), pares = superior (colunas, U22 e R52-R59), tudo medido.
- CN2 = entrada da fonte na placa principal.
- R30 é o pull-up do /HALT e R29 o do /IRQ; /OE da EPROM e das duas
  µPD41416 no GND (medidos).
- Roteiro de continuidade: 38 redes medidas, 6 parciais, 39 só da revista.
  Docs (hardware, teclado, origem) atualizados.

Co-Authored-By: Claude Opus 5.5 <noreply@anthropic.com>
Other:
- added sheet Fonte (fonte.kicad_sch)
- note added: "Primeira versão: parte digital. A parte analógica (PLL, sincronismo, croma, mixer) ainda é um bloco. O circuito junta as medidas de continuidade feitas no aparelho com o "Build This Video Titler" (Radio-Electronics, nov./1985 a mar./1986), de onde o VET deriva (docs/origem.md). A folha Fonte traz a placa da fonte, levantada das fotos dos dois lados (referências 2xx provisórias)."
- note added: "Referências: U14, U15, U16, U21, U22, U23, D8, D10, D11, R26-R30, R48, R49, R52-R59 e CN1-CN3 são as da placa. U101-U104, T101, C101-C114, R103-R105 e #BLK1 são provisórias: as da placa não aparecem nas fotos. O campo "rev." de cada peça dá o equivalente na revista."
- note removed: "Primeira versão: parte digital. A parte analógica (PLL, sincronismo, croma, mixer) ainda é um bloco. O circuito junta as medidas de continuidade feitas no aparelho com o "Build This Video Titler" (Radio-Electronics, nov./1985 a mar./1986), de onde o VET deriva (docs/origem.md)."
- note removed: "Referências: U14, U15, U16, U21, U22, U23, D8, D10, D11, R26-R30, R48, R49 e R52-R59 foram lidas na placa (fotos). U101-U104, T101, C101-C114, R103-R105, CN2 e #BLK1 são provisórias: as da placa não aparecem nas fotos. O campo "rev." de cada peça dá o equivalente na revista."
Changed lines of the file:
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@@
 		)
 	)
-	(text "Primeira versão: parte digital. A parte analógica (PLL, sincronismo, croma, mixer) ainda é um bloco.\nO circuito junta as medidas de continuidade feitas no aparelho com o \"Build This Video Titler\"\n(Radio-Electronics, nov./1985 a mar./1986), de onde o VET deriva (docs/origem.md)."
+	(text "Primeira versão: parte digital. A parte analógica (PLL, sincronismo, croma, mixer) ainda é um bloco.\nO circuito junta as medidas de continuidade feitas no aparelho com o \"Build This Video Titler\"\n(Radio-Electronics, nov./1985 a mar./1986), de onde o VET deriva (docs/origem.md).\nA folha Fonte traz a placa da fonte, levantada das fotos dos dois lados (referências 2xx provisórias)."
 		(exclude_from_sim no)
 		(at 25.4 29.21 0)
@@
 		)
 	)
-	(text "Referências: U14, U15, U16, U21, U22, U23, D8, D10, D11, R26-R30, R48, R49 e R52-R59 foram lidas na\nplaca (fotos). U101-U104, T101, C101-C114, R103-R105, CN2 e #BLK1 são provisórias: as da placa\nnão aparecem nas fotos. O campo \"rev.\" de cada peça dá o equivalente na revista."
+	(text "Referências: U14, U15, U16, U21, U22, U23, D8, D10, D11, R26-R30, R48, R49, R52-R59 e CN1-CN3 são\nas da placa. U101-U104, T101, C101-C114, R103-R105 e #BLK1 são provisórias: as da placa\nnão aparecem nas fotos. O campo \"rev.\" de cada peça dá o equivalente na revista."
 		(exclude_from_sim no)
 		(at 25.4 71.12 0)
@@
 				)
 			)
+		)
+	)
+	(sheet
+		(at 317.5 127)
+		(size 71.12 22.86)
+		(exclude_from_sim no)
+		(in_bom yes)
+		(on_board yes)
+		(dnp no)
+		(stroke
+			(width 0)
+			(type solid)
+		)
+		(fill
+			(color 0 0 0 0.0000)
+		)
+		(property "Sheetname" "Fonte"
+			(at 317.5 126.24 0)
+			(effects
+				(font
+					(size 1.524 1.524)
+				)
+				(justify left bottom)
+			)
+		)
+		(property "Sheetfile" "fonte.kicad_sch"
+			(at 317.5 150.62 0)
+			(effects
+				(font
+					(size 1.27 1.27)
+				)
+				(justify left top)
+			)
+		)
+		(instances
+			(project "vet3000_placa"
+				(path "/5e7a3000-0c4a-4e0c-9a11-00000000b0a1"
+					(page "7")
+				)
+			)
