File: hardware/placa-principal/video.kicad_sch (KiCad schematic)
At the start: 14 parts, among them T101 2N3906, U104 TMS9128NL, U14 uPD41416C-15, U21 uPD41416C-15

Commit message: Esquema: placa da fonte e medidas do teclado, pull-ups e /OE
- Folha Fonte (fonte.kicad_sch), levantada das fotos dos dois lados da
  placa: ponte com derivação central, 7805, 7812, 7905 com bomba de carga,
  backup da RAM (+3V_BAT) e conector de saída. Explica os ~11 V no +5 V
  quando a fonte é testada sem carga.
- Teclado medido: U16 (74LS273) e U22 (74LS244) ligam D0-D7 com os mesmos
  pinos da revista (Fig. 14), e o /CLR do U16 vai ao +5 V. O conector das
  membranas é o CN3: pino 1 embaixo à esquerda, ímpares = membrana inferior
  (linhas, U16), pares = superior (colunas, U22 e R52-R59), tudo medido.
- CN2 = entrada da fonte na placa principal.
- R30 é o pull-up do /HALT e R29 o do /IRQ; /OE da EPROM e das duas
  µPD41416 no GND (medidos).
- Roteiro de continuidade: 38 redes medidas, 6 parciais, 39 só da revista.
  Docs (hardware, teclado, origem) atualizados.

Co-Authored-By: Claude Opus 5.5 <noreply@anthropic.com>
Other:
- note added: "VRAM (Fig. 10 da revista): AD0-AD7 do VDP vão a A7-A0 das DRAMs, RD0-RD3 a uma e RD4-RD7 à outra; /OE das DRAMs no GND (medido). Qual das duas é U14 e qual é U21 não foi verificado."
- note removed: "VRAM (Fig. 10 da revista): AD0-AD7 do VDP vão a A7-A0 das DRAMs, RD0-RD3 a uma e RD4-RD7 à outra; /OE das DRAMs no GND. Qual das duas é U14 e qual é U21 não foi verificado."
Changed lines of the file:
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@@
 		)
 	)
-	(text "VRAM (Fig. 10 da revista): AD0-AD7 do VDP vão a A7-A0 das DRAMs,\nRD0-RD3 a uma e RD4-RD7 à outra; /OE das DRAMs no GND.\nQual das duas é U14 e qual é U21 não foi verificado."
+	(text "VRAM (Fig. 10 da revista): AD0-AD7 do VDP vão a A7-A0 das DRAMs,\nRD0-RD3 a uma e RD4-RD7 à outra; /OE das DRAMs no GND (medido).\nQual das duas é U14 e qual é U21 não foi verificado."
 		(exclude_from_sim no)
 		(at 304.8 20.32 0)
@@
 		)
 	)
-	(wire
-		(pts
-			(xy 25.4 208.28) (xy 25.4 213.36)
-		)
-		(stroke
-			(width 0)
-			(type default)
-		)
-	)
 	(global_label "VDP_CLK"
 		(shape passive)
@@
 					(unit 1)
 				)
-			)
-		)
-	)
-	(symbol
-		(lib_id "power:PWR_FLAG")
-		(at 25.4 208.28 0)
-		(unit 1)
-		(body_style 1)
-		(exclude_from_sim no)
-		(in_bom no)
-		(on_board no)
-		(in_pos_files no)
-		(dnp no)
-		(property "Reference" "#FLG01"
-			(at 25.4 205.74 0)
-			(show_name no)
-			(do_not_autoplace no)
-			(effects
-				(font
-					(size 1.27 1.27)
-				)
-				(hide yes)
-			)
-		)
-		(property "Value" "PWR_FLAG"
-			(at 25.4 204.47 0)
-			(show_name no)
-			(do_not_autoplace no)
-			(effects
-				(font
-					(size 1.27 1.27)
-				)
-			)
-		)
-		(property "Footprint" ""
-			(at 25.4 208.28 0)
-			(show_name no)
-			(do_not_autoplace no)
-			(effects
-				(font
-					(size 1.27 1.27)
-				)
-				(hide yes)
-			)
-		)
-		(property "Datasheet" ""
-			(at 25.4 208.28 0)
-			(show_name no)
-			(do_not_autoplace no)
-			(effects
-				(font
-					(size 1.27 1.27)
-				)
-				(hide yes)
-			)
-		)
-		(property "Description" ""
-			(at 25.4 208.28 0)
-			(show_name no)
-			(do_not_autoplace no)
-			(effects
-				(font
-					(size 1.27 1.27)
-				)
-				(hide yes)
-			)
-		)
-		(pin "1"
-		)
-		(instances
-			(project "vet3000_placa"
-				(path "/5e7a3000-0c4a-4e0c-9a11-00000000b0a1/c249e328-e554-5115-9836-355c77444dee"
-					(reference "#FLG01")
-					(unit 1)
-				)
-			)
-		)
-	)
-	(symbol
-		(lib_id "power:+12V")
-		(at 25.4 213.36 180)
-		(unit 1)
-		(body_style 1)
-		(exclude_from_sim no)
-		(in_bom no)
-		(on_board no)
-		(in_pos_files no)
-		(dnp no)
-		(property "Reference" "#PWR031"
-			(at 25.4 213.36 0)
-			(show_name no)
-			(do_not_autoplace no)
-			(effects
-				(font
-					(size 1.27 1.27)
-				)
-				(hide yes)
-			)
-		)
-		(property "Value" "+12V"
-			(at 25.4 218.44 0)
-			(show_name no)
-			(do_not_autoplace no)
-			(effects
-				(font
-					(size 1.27 1.27)
-				)
-			)
-		)
-		(property "Footprint" ""
-			(at 25.4 213.36 0)
-			(show_name no)
-			(do_not_autoplace no)
-			(effects
-				(font
-					(size 1.27 1.27)
-				)
-				(hide yes)
-			)
-		)
-		(property "Datasheet" ""
-			(at 25.4 213.36 0)
-			(show_name no)
-			(do_not_autoplace no)
-			(effects
-				(font
-					(size 1.27 1.27)
-				)
-				(hide yes)
-			)
-		)
-		(property "Description" ""
-			(at 25.4 213.36 0)
-			(show_name no)
-			(do_not_autoplace no)
-			(effects
-				(font
-					(size 1.27 1.27)
-				)
-				(hide yes)
-			)
-		)
-		(pin "1"
-		)
-		(instances
-			(project "vet3000_placa"
-				(path "/5e7a3000-0c4a-4e0c-9a11-00000000b0a1/c249e328-e554-5115-9836-355c77444dee"
-					(reference "#PWR031")
-					(unit 1)
-				)
