File: hardware/placa-principal/fonte.kicad_sch (KiCad schematic)
At the start: 32 parts, among them CN201 Saída para a placa principal, T201 LIDER, 19,75 VAC com CT (medi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, U201 LM340T-5 (7805), U202 7812, U203 7905

Commit message: Placa principal: CN2 e seleção do teclado medidos, fonte consertada
- CN2 medido: ordem inversa da do CN201 da fonte (GND no pino 1, -5 V no
  pino 5). Esquema, roteiro e docs corrigidos.
- Seleção do teclado medida: U15 pino 10 no clock do U16 e pino 9 nos
  enables do U22, como na revista. Roteiro: 40 redes medidas, 6 parciais,
  37 só da revista.
- Fonte: D210 identificado (1N4148, estava aberto); trocados D207, D208,
  D210, C203, C205 e R201. Tabela com as tensões medidas depois do
  conserto e carga de teste corrigida para 47 ohms (a de 100 ohms puxa
  menos que os ~60 mA do R201). O VET liga e mostra a abertura.

Trabalho feito em outra sessão, commitado sem alterações.

Co-Authored-By: Claude Opus 5.5 <noreply@anthropic.com>
Parts:
- D210: value 1N? (vidro) -> 1N4148; Nota vidro vermelho, em pé ao lado do cerâmico C211 -> vidro, em pé ao lado do cerâmico C211
Other:
- note added: "CN201 na ordem da etiqueta do gabinete: -5 V, +5 V, +3 V BAT, +12 V e GND (fio preto). Na placa, o +5V chega ao pino 2 por um jumper de fio. No CN2 da placa principal, a ordem é a inversa."
- note removed: "CN201 na ordem da etiqueta do gabinete: -5 V, +5 V, +3 V BAT, +12 V e GND (fio preto). Na placa, o +5V chega ao pino 2 por um jumper de fio."
Changed lines of the file:
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@@
 		)
 	)
-	(text "Backup da RAM (+3V_BAT): ligado, vem de BKP_ALIM por D207; desligado, das pilhas por D208. D210 prende\nBKP_ALIM uma queda de diodo acima do +5V (~5,6 V), e assim a RAM recebe ~5 V. A corrente de R201\n(~60 mA, ~0,5 W no resistor) passa por D210 e entra na linha de +5V. Sem carga no +5V (placa principal\ndesligada), ela não tem para onde ir, porque o 7805 não absorve corrente: a linha sobe a ~11 V.\nTeste a fonte com carga. Se D210 abrir, o +5V fica normal, mas o +3V_BAT sobe a ~12 V."
+	(text "Backup da RAM (+3V_BAT): ligado, vem de BKP_ALIM por D207; desligado, das pilhas por D208. D210 prende\nBKP_ALIM uma queda de diodo acima do +5V (~5,6 V), e assim a RAM recebe ~5 V. A corrente de R201\n(~60 mA, ~0,5 W no resistor) passa por D210 e entra na linha de +5V. Sem carga no +5V (placa principal\ndesligada), ela não tem para onde ir, porque o 7805 não absorve corrente: a linha sobe a ~11 V.\nTeste com carga acima de ~70 mA (47 ohms). Se D210 abrir, o +5V fica normal e o +3V_BAT vai a ~12 V."
 		(exclude_from_sim no)
 		(at 25.4 256.54 0)
@@
 		)
 	)
-	(text "CN201 na ordem da etiqueta do gabinete:\n-5 V, +5 V, +3 V BAT, +12 V e GND (fio preto).\nNa placa, o +5V chega ao pino 2 por um jumper de fio."
+	(text "CN201 na ordem da etiqueta do gabinete:\n-5 V, +5 V, +3 V BAT, +12 V e GND (fio preto).\nNa placa, o +5V chega ao pino 2 por um jumper de fio.\nNo CN2 da placa principal, a ordem é a inversa."
 		(exclude_from_sim no)
 		(at 317.5 149.86 0)
@@
 			)
 		)
-		(property "Value" "1N? (vidro)"
+		(property "Value" "1N4148"
 			(at 78.74 228.6 0)
 			(show_name no)
@@
 			)
 		)
-		(property "Nota" "vidro vermelho, em pé ao lado do cerâmico C211"
+		(property "Nota" "vidro, em pé ao lado do cerâmico C211"
 			(at 78.74 231.14 0)
 			(show_name no)
